File: SensorExtentionBoard/HallEffect.sch (KiCad schematic (older format))
At the start: 0 parts

Commit message: Added Hall Effect sensor test circuit
Parts:
- added J? (x3): Conn_01x03_Male, symbol Connector:Conn_01x03_Male
- added R? (x6): R, symbol Device:R
- added U?: ADS1015IDGS, Package_SO:TSSOP-10_3x3mm_P0.5mm, symbol Analog_ADC:ADS1015IDGS
Connections:
- new net: R?.1, R?.2, U?.4 (AIN0)
- new net: R?.1, R?.2, U?.5 (AIN1)
- new net: R?.1, R?.2, U?.6 (AIN2)
- new net +5V: U?.8 (VDD)
- new net GND: J?.3 (Pin_3), J?.3 (Pin_3), J?.3 (Pin_3), R?.2, R?.2, R?.2, U?.1 (ADDR), U?.3 (GND)
- new net HE0: J?.2 (Pin_2)
- new net HE0_VIN: J?.1 (Pin_1), R?.1
- new net HE1: J?.2 (Pin_2)
- new net HE1_VIN: J?.1 (Pin_1), R?.1
- new net HE2: J?.2 (Pin_2)
- new net HE2_VIN: J?.1 (Pin_1), R?.1
- new net HE_ADC_ALERT_~RDY: U?.2 (ALERT/RDY)
- new net HE_ADC_SCL: U?.10 (SCL)
- new net HE_ADC_SDA: U?.9 (SDA)
