File: SensorExtentionBoard/Thermocouple.sch (KiCad schematic (older format))
At the start: 0 parts

Commit message: Added Hall Effect sensor test circuit
Parts:
- added J? (x2): Conn_01x02_Male, symbol Connector:Conn_01x02_Male
- added R? (x2): 768, symbol Device:R
- added R? (x2): 12, symbol Device:R
- added U?: MCP4728, Package_SO:MSOP-10_3x3mm_P0.5mm, symbol Analog_DAC:MCP4728
- added U? (x6): TS3A24159DGSR, Package_SO:TSSOP-10_3x3mm_P0.5mm, symbol Analog_Switch:TS3A24159DGSR
Connections:
- new net: R?.1, U?.6 (VOUTA)
- new net: R?.1, U?.7 (VOUTB)
- new net +5V: U?.1 (VCC), U?.1 (VCC), U?.1 (VDD)
- new net GND: R?.2, R?.2, U?.10 (VSS), U?.2, U?.2, U?.6 (GND), U?.6 (GND), U?.7, U?.7
- new net TC0: R?.1, R?.2, U?.10, U?.5
- new net TC0+: J?.1 (Pin_1), U?.3
- new net TC0-: J?.2 (Pin_2), U?.9
- new net TC0_Pol: U?.4, U?.8
- new net TC1: R?.1, R?.2, U?.10, U?.5
- new net TC1+: J?.1 (Pin_1), U?.3
- new net TC1-: J?.2 (Pin_2), U?.9
- new net TC1_Pol: U?.4, U?.8
- new net TC_RDY_~BSY: U?.5 (RDY/~BSY)
- new net TC_SCL: U?.2 (SCL)
- new net TC_SDA: U?.3 (SDA)
- new net TC_~LDAC: U?.4 (~LDAC)
- no-connect marks 0 -> 2
